Commit message: update 4

File: description/robot.urdf.xacro (robot description, xacro)
@@ -1,5 +1,4 @@
 <?xml version="1.0"?>
 <robot xmlns:xacro="http://www.ros.org/wiki/xacro"  name="Spot Micro">
-    <!-- Example link -->
-    <link name="base_link"></link>
+    <xacro:include filename="spot_core.xacro"/>
 </robot>
